Commit message: zzbzbzb

File: data/zzb/Take_022_Skeleton0_with_objtraj/shelf.urdf (robot description, URDF)
Before this commit: robot shelf, 1 links, 0 joints
Links:
- link shelf_link: geometry collision mesh filename=/Users/zbzhou/Documents/New project/shelf_compressed.obj scale=1 1 1; visual mesh filename=/Users/zbzhou/Documents/New project/shelf_compressed.obj scale=1 1 1

Commit message: dndndn

File: data/zzb/Take_022_Skeleton0_with_objtraj/shelf.urdf (robot description, URDF)
Before this commit: robot shelf_compressed, 1 links, 0 joints
Links:
- link shelf_link: geometry collision mesh filename=shelf.obj scale=1 1 1; visual mesh filename=shelf.obj scale=1 1 1
